File: Hardware/E-Load 2024.kicad_sch (KiCad schematic)
At the start: 73 parts, among them J1 Conn_01x06_Pin, Q1 NMOS, Q2 NMOS, U1 LM358, U2 ACS71240LLCBTR-010B3, U3 ACS71240LLCBTR-010B3, U4 MCP4725xxx-xCH, U5 ADS1115IDGS

Commit message: Load PCB is missing 3V3
Parts:
- removed TP15: VIN2, TestPoint:TestPoint_Pad_D2.5mm, symbol Connector:TestPoint_Alt
- removed TP2: VIN1, TestPoint:TestPoint_Pad_D2.5mm, symbol Connector:TestPoint_Alt
- added C11: 100nF, Capacitor_SMD:C_0805_2012Metric, symbol Device:C_Small
- added JP7: A0, Jumper:SolderJumper-2_P1.3mm_Open_RoundedPad1.0x1.5mm, symbol Jumper:SolderJumper_2_Open
- added JP8: A1, Jumper:SolderJumper-2_P1.3mm_Open_RoundedPad1.0x1.5mm, symbol Jumper:SolderJumper_2_Open
- added JP9: A2, Jumper:SolderJumper-2_P1.3mm_Open_RoundedPad1.0x1.5mm, symbol Jumper:SolderJumper_2_Open
- added R17, R18, R19: 10k, Resistor_SMD:R_0805_2012Metric, symbol Device:R_Small
- added U6: 24LC32, Package_SO:SOIC-8_3.9x4.9mm_P1.27mm, symbol Memory_EEPROM:24LC32
- H1, H2, H3, H4: symbol Mechanical:MountingHole_Pad_MP -> Mechanical:MountingHole_Pad
- U1: footprint Package_SO:SOIC-8_3.9x4.9mm_P1.27mm -> Package_SO:TSSOP-8_4.4x3mm_P0.65mm
- U5: footprint Package_SO:TSSOP-10_3x3mm_P0.5mm -> Package_SO:VSSOP-10_3x3mm_P0.5mm
Connections:
- net +3V3: now also C11.1, JP7.2 (B), JP8.2 (B), JP9.2 (B), U6.8 (VCC)
- net -VDC: now also H3.1, H4.1, C11.2, R17.2, R18.2, R19.2, U6.4 (GND), U6.7 (WP); no longer H3.MP, H4.MP
- net SCL: now also U6.6 (SCL)
- net SDA: now also U6.5 (SDA)
- net VIN1: now also F1.2, Q1.1 (D); no longer F1.1, H1.MP
- net VIN2: now also F2.2, Q2.1 (D); no longer F2.1, H2.MP
- new net: JP8.1 (A), R18.1, U6.2 (A1)
- new net: F2.1, H2.1
- new net: JP7.1 (A), R17.1, U6.1 (A0)
- new net: JP9.1 (A), R19.1, U6.3 (A2)
- new net: F1.1, H1.1
Other:
- moved on the sheet: C1, C2, H3, H4, U1C
