File: Hardware/E-Load 2024.kicad_pcb (KiCad board)
At the start: 2 copper layers, 160 x 100 mm, 0 parts

Commit message: Load PCB is missing 3V3
Parts:
- added C1: 100nF, Capacitor_SMD:C_0805_2012Metric, F.Cu at (79.4, 88.8)
- added C10: 10uF T, Capacitor_SMD:C_1206_3216Metric, F.Cu at (74.3, 67.8)
- added C11: 100nF, Capacitor_SMD:C_0805_2012Metric, F.Cu at (188.2, 124.0)
- added C2: 100nF, Capacitor_SMD:C_0805_2012Metric, F.Cu at (82.3, 103.0)
- added C3: 100nF, Capacitor_SMD:C_0805_2012Metric, F.Cu at (98.8, 68.8)
- added C4: 220uF, Capacitor_SMD:CP_Elec_6.3x5.8, F.Cu at (82.8, 126.1)
- added C5: 100nF, Capacitor_SMD:C_0805_2012Metric, F.Cu at (109.6, 128.5)
- added C6: 100nF, Capacitor_SMD:C_0805_2012Metric, F.Cu at (74.2, 70.7)
- added C7: 100nF, Capacitor_SMD:C_0805_2012Metric, F.Cu at (74.6, 106.2)
- added C8: 10uF T, Capacitor_SMD:C_1206_3216Metric, F.Cu at (74.5, 103.0)
- added C9: 220uF, Capacitor_SMD:CP_Elec_6.3x5.8, F.Cu at (64.3, 97.4)
- added D1: LED, LED_SMD:LED_0805_2012Metric, F.Cu at (205.7, 102.3)
- added D2: LED, LED_SMD:LED_0805_2012Metric, F.Cu at (205.7, 93.5)
- added D3: 1N4148, Diode_SMD:D_SOD-323, F.Cu at (101.6, 111.1)
- added D4: 1N4148, Diode_SMD:D_SOD-323, F.Cu at (101.7, 107.7)
- added D5: 1N4148, Diode_SMD:D_SOD-323, F.Cu at (101.8, 85.4)
- added D6: 1N4148, Diode_SMD:D_SOD-323, F.Cu at (101.8, 88.4)
- added F1: 7,5A, Fuseholder:BX503-35, F.Cu at (65.5, 142.2)
- added F2: 7,5A, Fuseholder:BX503-35, F.Cu at (66.6, 58.4)
- added H1: IN_MOS1, MountingHole:MountingHole_5.3mm_M5_Pad_Via, F.Cu at (86.1, 142.2)
- added H2: IN_MOS2, MountingHole:MountingHole_5.3mm_M5_Pad_Via, F.Cu at (86.1, 58.1)
- added H3: GND, MountingHole:MountingHole_5.3mm_M5_Pad_Via, F.Cu at (148.4, 58.1)
- added H4: GND, MountingHole:MountingHole_5.3mm_M5_Pad_Via, F.Cu at (148.4, 142.2)
- added J1: Conn_01x06_Pin, Connector_JST:JST_XH_B8B-XH-A_1x08_P2.50mm_Vertical, F.Cu at (200.7, 76.0)
- added JP1: SolderJumper_2_Open, Jumper:SolderJumper-2_P1.3mm_Open_RoundedPad1.0x1.5mm, F.Cu at (116.8, 121.3)
- added JP2: SolderJumper_2_Open, Jumper:SolderJumper-2_P1.3mm_Open_RoundedPad1.0x1.5mm, F.Cu at (116.8, 124.8)
- added JP3: SolderJumper_2_Open, Jumper:SolderJumper-2_P1.3mm_Open_RoundedPad1.0x1.5mm, F.Cu at (114.1, 74.9)
- added JP4: SolderJumper_2_Open, Jumper:SolderJumper-2_P1.3mm_Open_RoundedPad1.0x1.5mm, F.Cu at (114.1, 71.4)
- added JP5: SolderJumper_2_Open, Jumper:SolderJumper-2_P1.3mm_Open_RoundedPad1.0x1.5mm, F.Cu at (114.1, 67.8)
- added JP6: SolderJumper_2_Open, Jumper:SolderJumper-2_P1.3mm_Open_RoundedPad1.0x1.5mm, F.Cu at (114.1, 64.3)
- added JP7: A0, Jumper:SolderJumper-2_P1.3mm_Open_RoundedPad1.0x1.5mm, F.Cu at (186.9, 141.4)
- added JP8: A1, Jumper:SolderJumper-2_P1.3mm_Open_RoundedPad1.0x1.5mm, F.Cu at (191.3, 141.4)
- added JP9: A2, Jumper:SolderJumper-2_P1.3mm_Open_RoundedPad1.0x1.5mm, F.Cu at (195.7, 141.4)
- added Q1: NMOS, Package_TO_SOT_THT:TO-247-3_Vertical, F.Cu at (56.1, 125.2)
- added Q2: NMOS, Package_TO_SOT_THT:TO-247-3_Vertical, F.Cu at (56.1, 90.0)
- added R1: 22k, Resistor_SMD:R_0805_2012Metric, F.Cu at (89.2, 103.5)
- added R10: 330, Resistor_SMD:R_0805_2012Metric, F.Cu at (205.7, 89.5)
- added R11: 10k, Resistor_SMD:R_0805_2012Metric, F.Cu at (66.0, 84.6)
- added R12: 20m, Resistor_SMD:R_1210_3225Metric_Pad1.30x2.65mm_HandSolder, F.Cu at (65.1, 79.0)
- added R13: 10k, Resistor_SMD:R_0805_2012Metric, F.Cu at (199.9, 89.5)
- added R14: 0, Resistor_SMD:R_0805_2012Metric, F.Cu at (101.8, 94.3)
- added R15: 8.2k, Resistor_SMD:R_0805_2012Metric, F.Cu at (101.7, 114.7)
- added R16: 8.2k, Resistor_SMD:R_0805_2012Metric, F.Cu at (101.9, 81.9)
- added R17: 10k, Resistor_SMD:R_0805_2012Metric, F.Cu at (186.9, 147.5)
- added R18: 10k, Resistor_SMD:R_0805_2012Metric, F.Cu at (191.3, 147.5)
- added R19: 10k, Resistor_SMD:R_0805_2012Metric, F.Cu at (195.7, 147.4)
- added R2: 100, Resistor_SMD:R_0805_2012Metric, F.Cu at (91.1, 125.2)
- added R3: 10k, Resistor_SMD:R_0805_2012Metric, F.Cu at (66.0, 119.8)
- added R4: 20m, Resistor_SMD:R_1210_3225Metric_Pad1.30x2.65mm_HandSolder, F.Cu at (65.1, 114.2)
- added R5: 22k, Resistor_SMD:R_0805_2012Metric, F.Cu at (89.2, 86.5)
- added R6: 10k, Resistor_SMD:R_0805_2012Metric, F.Cu at (199.9, 106.3)
- added R7: 0, Resistor_SMD:R_0805_2012Metric, F.Cu at (101.8, 101.8)
- added R8: 330, Resistor_SMD:R_0805_2012Metric, F.Cu at (205.7, 106.3)
- added R9: 100, Resistor_SMD:R_0805_2012Metric, F.Cu at (61.6, 103.7)
- added RV1: 1k, Potentiometer_THT:Potentiometer_Bourns_3296W_Vertical, F.Cu at (90.0, 98.2)
- added RV2: 1k, Potentiometer_THT:Potentiometer_Bourns_3296W_Vertical, F.Cu at (90.0, 92.3)
- added RV3: 1k, Potentiometer_THT:Potentiometer_Bourns_3296W_Vertical, F.Cu at (106.4, 101.8)
- added RV4: 1k, Potentiometer_THT:Potentiometer_Bourns_3296W_Vertical, F.Cu at (106.4, 94.3)
- added RV5: 1k, Potentiometer_THT:Potentiometer_Bourns_3296W_Vertical, F.Cu at (106.4, 109.1)
- added RV6: 1k, Potentiometer_THT:Potentiometer_Bourns_3296W_Vertical, F.Cu at (106.4, 87.1)
- added TP1: VCTRL_1, TestPoint:TestPoint_Pad_D2.5mm, F.Cu at (93.2, 104.4)
- added TP10: GND, TestPoint:TestPoint_Pad_D2.5mm, F.Cu at (191.1, 65.5)
- added TP11: ACS2_OUT, TestPoint:TestPoint_Pad_D2.5mm, F.Cu at (107.3, 75.9)
- added TP12: -12V, TestPoint:TestPoint_Pad_D2.5mm, F.Cu at (191.1, 59.7)
- added TP13: +12V, TestPoint:TestPoint_Pad_D2.5mm, F.Cu at (191.1, 53.8)
- added TP14: V_CTRL, TestPoint:TestPoint_Pad_D2.5mm, F.Cu at (84.2, 85.2)
- added TP3: OA1_O, TestPoint:TestPoint_Pad_D2.5mm, F.Cu at (82.2, 112.9)
- added TP4: VCTRL_2, TestPoint:TestPoint_Pad_D2.5mm, F.Cu at (94.5, 86.5)
- added TP5: ACS1_OUT, TestPoint:TestPoint_Pad_D2.5mm, F.Cu at (116.7, 101.9)
- added TP6: OA2_O, TestPoint:TestPoint_Pad_D2.5mm, F.Cu at (84.2, 90.0)
- added TP7: SDA, TestPoint:TestPoint_Pad_D2.5mm, F.Cu at (191.1, 77.1)
- added TP8: SCL, TestPoint:TestPoint_Pad_D2.5mm, F.Cu at (191.1, 82.9)
- added TP9: 3V3, TestPoint:TestPoint_Pad_D2.5mm, F.Cu at (191.1, 71.3)
- added U1: LM358, Package_SO:TSSOP-8_4.4x3mm_P0.65mm, F.Cu at (80.4, 96.0)
- added U2: ACS71240LLCBTR-010B3, Package_SO:SOIC-8_3.9x4.9mm_P1.27mm, F.Cu at (75.1, 111.8)
- added U3: ACS71240LLCBTR-010B3, Package_SO:SOIC-8_3.9x4.9mm_P1.27mm, F.Cu at (73.9, 76.6)
- added U4: MCP4725xxx-xCH, Package_TO_SOT_SMD:SOT-23-6, F.Cu at (109.5, 122.9)
- added U5: ADS1115IDGS, Package_SO:VSSOP-10_3x3mm_P0.5mm, F.Cu at (104.3, 69.3)
- added U6: 24LC32, Package_SO:SOIC-8_3.9x4.9mm_P1.27mm, F.Cu at (189.4, 131.4)
Routing:
- net SCL: track 0.00 -> 279.2 mm, vias 0 -> 6
- net SDA: track 0.00 -> 258.5 mm, vias 0 -> 3
- net -12V: track 0.00 -> 165.3 mm, vias 0 -> 4
- net +12V: track 0.00 -> 158.3 mm, vias 0 -> 2
- net FAULT2: track 0.00 -> 137.9 mm, vias 0 -> 4
- net FAULT1: track 0.00 -> 134.1 mm, vias 0 -> 2
- net D_RDY: track 0.00 -> 110.8 mm, vias 0 -> 1
- net VIN2: track 0.00 -> 93.4 mm, vias 0 -> 1
- net -VDC: track 0.00 -> 91.8 mm, vias 0 -> 33
- net VIN1: track 0.00 -> 72.1 mm, vias 0 -> 1
- net V_SENSE1: track 0.00 -> 60.3 mm, vias 0 -> 3
- net V_CTRL: track 0.00 -> 56.1 mm, vias 0 -> 4
- net Net-(C4-Pad1): track 0.00 -> 55.3 mm
- net C1: track 0.00 -> 47.4 mm
- net +3V3: track 0.00 -> 47.2 mm
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- added copper zone on B.Cu, net -VDC
- added copper zone on F.Cu, net -VDC
- added copper zone on F.Cu, net Net-(Q1-S)
- added copper zone on F.Cu, net Net-(Q2-S)
- added copper zone on F.Cu, net Net-(R12-Pad2)
- added copper zone on F.Cu, net Net-(R4-Pad2)

Commit message: Final Version 1.0
Parts:
- added M3_1: MountingHole_3.2mm_M3_DIN965, MountingHole:MountingHole_3.2mm_M3_DIN965, F.Cu at (125.0, 65.0)
- added M3_2: MountingHole_3.2mm_M3_DIN965, MountingHole:MountingHole_3.2mm_M3_DIN965, F.Cu at (55.0, 100.0)
- added M3_3: MountingHole_3.2mm_M3_DIN965, MountingHole:MountingHole_3.2mm_M3_DIN965, F.Cu at (125.0, 135.0)
- moved D1 59.2 mm to (146.6, 102.0)
- moved D2 59.2 mm to (146.6, 93.2)
- moved R10 59.2 mm to (146.6, 89.2)
- moved R8 59.2 mm to (146.6, 106.0)
- moved R13 59.2 mm to (140.7, 89.2)
- moved R6 59.2 mm to (140.7, 106.0)
- moved R18 55.8 mm to (135.6, 146.1)
- moved R17 55.8 mm to (131.2, 146.1)
- moved R19 55.8 mm to (140.0, 146.0)
- moved JP8 55.8 mm to (135.6, 141.1)
- moved C11 55.8 mm to (132.4, 123.7)
- moved J1 55.8 mm to (144.9, 75.7)
- moved JP7 55.8 mm to (131.2, 141.1)
- moved JP9 55.8 mm to (140.0, 141.1)
- moved TP10 55.8 mm to (135.4, 65.2)
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Routing:
- net +3V3: track 47.2 -> 337.6 mm, vias 0 -> 4
- net SCL: track 279.2 -> 176.2 mm, vias 6 -> 2
- net SDA: track 258.5 -> 178.7 mm, vias 3 -> 1
- net -12V: track 165.3 -> 88.6 mm, vias 4 -> 0
- net D_RDY: track 110.8 -> 44.2 mm, vias 1 -> 2
- net FAULT1: track 134.1 -> 74.1 mm, vias 2 -> 0
- net +12V: track 158.3 -> 101.0 mm
- net -VDC: track 91.8 -> 41.8 mm, vias 33 -> 43
- net VIN2: track 93.4 -> 49.4 mm, vias 1 -> 42
- net FAULT2: track 137.9 -> 94.4 mm, vias 4 -> 2
- net VIN1: track 72.1 -> 53.6 mm, vias 1 -> 14
- net Net-(F2-Pad1): track 17.5 -> 0.00 mm
- net Net-(F1-Pad1): track 18.5 -> 25.6 mm, vias 0 -> 5
- net Net-(C9-Pad1): track 42.2 -> 35.1 mm
- net Net-(JP3-B): track 24.7 -> 31.7 mm
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- added copper zone on B.Cu, net Net-(F1-Pad1)
- added copper zone on F.Cu, net Net-(F1-Pad1)
- added copper zone on B.Cu, net Net-(F2-Pad1)
- added copper zone on F.Cu, net Net-(F2-Pad1)
- added copper zone on B.Cu, net Net-(Q1-S)
- added copper zone on B.Cu, net Net-(Q2-S)
- added copper zone on B.Cu, net Net-(R12-Pad2)
- added copper zone on B.Cu, net Net-(R4-Pad2)
- added copper zone on B.Cu, net VIN1
- added copper zone on F.Cu, net VIN1
- added copper zone on B.Cu, net VIN2
- added copper zone on F.Cu, net VIN2
Other:
- board size 160 x 100 mm -> 100 x 100 mm
- board text added: "GND"
- board text added: "VIN1"
- board text added: "VIN2"
